File: circuit-board/v2-scratch.sch (EAGLE design)
At the start: 50 parts, among them IC1 UA78M05DCY, Q1 BC547B, Q2 BC547B, U1 MAX3232, U2 ATMEGA328P_TQFP, U3 ADUM1201BRZ, Y1 16MHz

Commit message: Clean up circuit diagrams, prep for prototype
Parts:
- added 12V-IN-HDST: JST-XH-02-PIN-LONG-PAD, Rembrandt Electronics - JST XH Connectors v1-0:JST-XH-02-PIN-LONG-PAD
- added R6: 220, SparkFun-Resistors:220OHM-0603-1/10W-1%
- added R9: 1k, SparkFun-Resistors:1KOHM-0603-1/10W-1%
- renumbered 12V-IN to 12V-IN-GPS
Connections:
- new net N$8: C21.+, R8.1
- new net N$9: OK1.A, R6.1
- new net RADIO-PTT-SENSE: OK1.COL, R4.2
- net 12V: now also 12V-IN-HDST-2.S, R6.2, R9.2; no longer R8.2
- net GND: now also OK1.EMI
- net GNDA: now also 12V-IN-HDST-1.S
- net HANDSET-PTT: now also OK1.C; no longer R4.1
- net RADIO-MIC/PTT: now also R4.1; no longer R4.2
- net RADIO-SPK-OUT: now also R8.2; no longer C21.+
- net SPKAMP: now also R9.1; no longer R8.1
Other:
- moved on the sheet: C1, C16, C17, C18, C19, C2, C20, C21, C5, C9, FB1, IC1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
