File: circuit-board/circuit-board.brd (EAGLE design)
At the start: 50.8 x 45.7 mm, 53 parts, among them IC1 UA78M05DCY, Q1 BC547B, Q2 BC547B, U1 MAX3232, U2 ATMEGA328P, U3 ADUM1201BRZ, Y2 16MHz

Commit message: Eliminate overlapping parts in V2 board layout
Parts:
- moved C20 2.41 mm to (2.79, 26.8)
- moved C2 1.91 mm to (41.4, 35.8)
- moved EXP-GND 1.28 mm to (46.4, 34.7)
- moved R9 1.17 mm to (37.5, 37.8)
- moved C16 1.05 mm to (4.57, 42.7)
- moved EXT-GND 0.46 mm to (49.1, 34.7)
Routing:
- net N$1: track 13.9 -> 15.1 mm
- net N$10: track 2.07 -> 3.18 mm
- net N$5: track 9.31 -> 10.3 mm
- net +5V: track 78.1 -> 79.1 mm
- net N$2: track 3.05 -> 3.59 mm
Changed lines of the file:
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@@
 <attribute name="VALUE" x="18.288" y="5.08" size="0.6096" layer="25" font="vector" ratio="20" rot="R180" align="top-center"/>
 </element>
-<element name="C16" library="adafruit" library_urn="urn:adsk.eagle:library:420" package="E2,5-5" value="10uF" x="4.318" y="41.656" smashed="yes">
-<attribute name="VALUE" x="3.429" y="44.45" size="0.6096" layer="25" ratio="10"/>
+<element name="C16" library="adafruit" library_urn="urn:adsk.eagle:library:420" package="E2,5-5" value="10uF" x="4.572" y="42.672" smashed="yes">
+<attribute name="VALUE" x="7.874" y="42.164" size="0.6096" layer="25" ratio="10" rot="R90"/>
 </element>
 <element name="C17" library="SparkFun-Capacitors" package="0603" value="0.1uF" x="3.937" y="39.116" smashed="yes">
@@
 <attribute name="VALUE" x="1.27" y="30.226" size="0.6096" layer="25" font="vector" ratio="20" rot="R90" align="top-center"/>
 </element>
-<element name="C2" library="adafruit" library_urn="urn:adsk.eagle:library:420" package="E2,5-5" value="10uF" x="39.497" y="35.814" smashed="yes" rot="R270">
-<attribute name="VALUE" x="40.894" y="38.227" size="0.6096" layer="25" ratio="10"/>
-</element>
-<element name="C20" library="adafruit" library_urn="urn:adsk.eagle:library:420" package="E2,5-5" value="10uF" x="5.08" y="27.559" smashed="yes">
-<attribute name="VALUE" x="8.509" y="26.797" size="0.6096" layer="25" ratio="10" rot="R90"/>
+<element name="C2" library="adafruit" library_urn="urn:adsk.eagle:library:420" package="E2,5-5" value="10uF" x="41.402" y="35.814" smashed="yes" rot="R270">
+<attribute name="VALUE" x="42.799" y="38.227" size="0.6096" layer="25" ratio="10"/>
+</element>
+<element name="C20" library="adafruit" library_urn="urn:adsk.eagle:library:420" package="E2,5-5" value="10uF" x="2.794" y="26.797" smashed="yes">
+<attribute name="VALUE" x="5.588" y="28.575" size="0.6096" layer="25" ratio="10" rot="R270"/>
 </element>
 <element name="C21" library="adafruit" library_urn="urn:adsk.eagle:library:420" package="E2,5-5" value="10uF" x="42.164" y="9.271" smashed="yes" rot="R90">
@@
 <attribute name="VALUE" x="40.386" y="11.811" size="0.6096" layer="25" ratio="10" rot="R180"/>
 </element>
-<element name="EXP-GND" library="SparkFun-Connectors" package="1X02" value="" x="45.085" y="34.798" rot="R90"/>
-<element name="EXT-GND" library="SparkFun-Connectors" package="1X02" value="" x="48.768" y="34.417" rot="R90"/>
+<element name="EXP-GND" library="SparkFun-Connectors" package="1X02" value="" x="46.355" y="34.671" rot="R90"/>
+<element name="EXT-GND" library="SparkFun-Connectors" package="1X02" value="" x="49.149" y="34.671" smashed="yes" rot="R90">
+<attribute name="NAME" x="49.657" y="33.147" size="0.6096" layer="25" font="vector" ratio="20" rot="R270"/>
+<attribute name="VALUE" x="51.181" y="33.401" size="0.6096" layer="27" font="vector" ratio="20" rot="R90"/>
+</element>
 <element name="FB1" library="SparkFun-Coils" package="0603" value="30Ω/1.8A" x="10.541" y="30.607" smashed="yes" rot="R180">
 <attribute name="NAME" x="10.541" y="29.845" size="0.6096" layer="25" font="vector" ratio="20" rot="R180" align="bottom-center"/>
@@
 <attribute name="VALUE" x="34.036" y="20.447" size="0.6096" layer="25" font="vector" ratio="20" align="top-center"/>
 </element>
-<element name="R9" library="SparkFun-Resistors" library_urn="urn:adsk.eagle:library:532" package="0603" package3d_urn="urn:adsk.eagle:package:39650/1" value="100" x="36.576" y="37.084" smashed="yes" rot="R180">
-<attribute name="PROD_ID" value="RES-07863" x="36.576" y="37.084" size="1.778" layer="27" rot="R180" display="off"/>
-<attribute name="VALUE" x="36.576" y="37.846" size="0.6096" layer="25" font="vector" ratio="20" rot="R180" align="top-center"/>
+<element name="R9" library="SparkFun-Resistors" library_urn="urn:adsk.eagle:library:532" package="0603" package3d_urn="urn:adsk.eagle:package:39650/1" value="100" x="37.465" y="37.846" smashed="yes" rot="R180">
+<attribute name="PROD_ID" value="RES-07863" x="37.465" y="37.846" size="1.778" layer="27" rot="R180" display="off"/>
+<attribute name="VALUE" x="37.465" y="36.449" size="0.6096" layer="25" font="vector" ratio="20" rot="R180" align="top-center"/>
 </element>
 </elements>
@@
 <contactref element="HANDSET" pad="5"/>
 <contactref element="EXP-GND" pad="2"/>
-<wire x1="45.085" y1="37.338" x2="45.085" y2="41.402" width="0.1524" layer="1"/>
-<wire x1="45.085" y1="41.402" x2="45.466" y2="41.783" width="0.1524" layer="1"/>
+<wire x1="45.466" y1="41.783" x2="45.466" y2="38.1" width="0.1524" layer="1"/>
+<wire x1="45.466" y1="38.1" x2="46.355" y2="37.211" width="0.1524" layer="1"/>
 </signal>
 <signal name="HANDSET-EXT">
 <contactref element="HANDSET" pad="6"/>
 <contactref element="EXT-GND" pad="2"/>
-<wire x1="48.006" y1="41.783" x2="48.768" y2="41.021" width="0.1524" layer="1"/>
-<wire x1="48.768" y1="41.021" x2="48.768" y2="36.957" width="0.1524" layer="1"/>
+<wire x1="48.006" y1="41.783" x2="48.006" y2="38.354" width="0.1524" layer="1"/>
+<wire x1="48.006" y1="38.354" x2="49.149" y2="37.211" width="0.1524" layer="1"/>
 </signal>
 <signal name="RADIO-MIC/PTT">
@@
 <wire x1="3.1242" y1="32.3596" x2="2.706" y2="31.9414" width="0.1524" layer="1"/>
 <wire x1="2.706" y1="31.9414" x2="2.706" y2="30.226" width="0.1524" layer="1"/>
-<wire x1="3.81" y1="27.559" x2="2.706" y2="28.663" width="0.1524" layer="1"/>
-<wire x1="2.706" y1="28.663" x2="2.706" y2="30.226" width="0.1524" layer="1"/>
 <wire x1="16.129" y1="19.265" x2="14.384" y2="17.52" width="0.1524" layer="1"/>
 <wire x1="14.384" y1="17.52" x2="14.224" y2="17.52" width="0.1524" layer="1"/>
@@
 <wire x1="11.811" y1="20.32" x2="5.715" y2="20.32" width="0.1524" layer="16"/>
 <via x="5.715" y="20.32" extent="1-16" drill="0.35"/>
-<wire x1="5.715" y1="20.32" x2="3.81" y2="22.225" width="0.1524" layer="1"/>
-<wire x1="3.81" y1="22.225" x2="3.81" y2="27.559" width="0.1524" layer="1"/>
 <wire x1="14.224" y1="17.52" x2="14.611" y2="17.52" width="0.1524" layer="1"/>
 <wire x1="14.611" y1="17.52" x2="16.383" y2="15.748" width="0.1524" layer="1"/>
@@
 <wire x1="11.43" y1="8.89" x2="12.9669125" y2="8.89" width="0.1524" layer="1"/>
 <wire x1="12.9669125" y1="8.89" x2="13.4689125" y2="9.392" width="0.1524" layer="1"/>
+<wire x1="2.706" y1="30.226" x2="2.706" y2="27.979" width="0.1524" layer="1"/>
+<wire x1="2.706" y1="27.979" x2="1.524" y2="26.797" width="0.1524" layer="1"/>
+<wire x1="1.524" y1="26.797" x2="1.524" y2="24.511" width="0.1524" layer="1"/>
+<wire x1="1.524" y1="24.511" x2="5.715" y2="20.32" width="0.1524" layer="1"/>
 </signal>
 <signal name="N$1">
@@
 <wire x1="3.3156" y1="36.9824" x2="3.1242" y2="36.9824" width="0.1524" layer="1"/>
 <wire x1="3.087" y1="39.116" x2="3.048" y2="39.155" width="0.1524" layer="1"/>
-<wire x1="3.048" y1="39.155" x2="3.048" y2="41.656" width="0.1524" layer="1"/>
+<wire x1="3.087" y1="39.116" x2="3.087" y2="42.457" width="0.1524" layer="1"/>
+<wire x1="3.087" y1="42.457" x2="3.302" y2="42.672" width="0.1524" layer="1"/>
 </signal>
 <signal name="SPKAMP">
@@
 <contactref element="C2" pad="-"/>
 <contactref element="SPK-XFMR" pad="6"/>
-<wire x1="39.497" y1="31.496" x2="39.497" y2="34.544" width="0.1524" layer="1"/>
+<wire x1="39.497" y1="31.496" x2="41.402" y2="34.544" width="0.1524" layer="1"/>
 </signal>
 <signal name="N$5">
@@
 <wire x1="30.099" y1="40.767" x2="27.94" y2="40.767" width="0.1524" layer="1"/>
 <contactref element="R9" pad="2"/>
-<wire x1="33.782" y1="37.084" x2="35.726" y2="37.084" width="0.1524" layer="1"/>
+<wire x1="33.782" y1="37.084" x2="36.615" y2="37.846" width="0.1524" layer="1"/>
 </signal>
 <signal name="N$6">
@@
 <contactref element="C2" pad="+"/>
 <contactref element="R9" pad="1"/>
-<wire x1="37.426" y1="37.084" x2="39.497" y2="37.084" width="0.1524" layer="1"/>
+<wire x1="38.315" y1="37.846" x2="41.402" y2="37.084" width="0.1524" layer="1"/>
 </signal>
 </signals>
