File: circuit-board/circuit-board.brd (EAGLE design)
At the start: 50.8 x 45.7 mm, 53 parts, among them IC1 UA78M05DCY, Q1 BC547B, Q2 BC547B, U1 MAX3232, U2 ATMEGA328P, U3 ADUM1201BRZ, Y2 16MHz

Commit message: Switched 100/120 ohm resistors in audio amp circuit for 1k resistors -- noise almost eliminated, though serial noise remains.. will need to split up ground planes to clear that up
Parts:
- R2: value 120 -> 1k
- R8, R9: value 100 -> 1k
Changed lines of the file:
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@@
 <?xml version="1.0" encoding="utf-8"?>
 <!DOCTYPE eagle SYSTEM "eagle.dtd">
-<eagle version="8.6.3">
+<eagle version="9.2.2">
 <drawing>
 <settings>
@@
 <param name="checkStop" value="0"/>
 <param name="checkValues" value="0"/>
+<param name="checkNames" value="1"/>
+<param name="checkWireStubs" value="1"/>
+<param name="checkPolygonWidth" value="0"/>
 <param name="useDiameter" value="13"/>
 <param name="maxErrors" value="50"/>
@@
 <attribute name="VALUE" x="40.386" y="11.811" size="0.6096" layer="25" ratio="10" rot="R180"/>
 </element>
-<element name="EXP-GND" library="SparkFun-Connectors" package="1X02" value="" x="46.355" y="34.671" rot="R90"/>
+<element name="EXP-GND" library="SparkFun-Connectors" package="1X02" value="" x="46.355" y="34.671" smashed="yes" rot="R90">
+<attribute name="NAME" x="44.958" y="33.401" size="0.6096" layer="25" font="vector" ratio="20" rot="R90"/>
+<attribute name="VALUE" x="48.387" y="33.401" size="0.6096" layer="27" font="vector" ratio="20" rot="R90"/>
+</element>
 <element name="EXT-GND" library="SparkFun-Connectors" package="1X02" value="" x="49.149" y="34.671" smashed="yes" rot="R90">
 <attribute name="NAME" x="49.657" y="33.147" size="0.6096" layer="25" font="vector" ratio="20" rot="R270"/>
@@
 <attribute name="VALUE" x="48.26" y="8.255" size="0.6096" layer="25" font="vector" ratio="20" rot="R180" align="top-center"/>
 </element>
-<element name="R2" library="SparkFun-Resistors" package="0603" value="120" x="33.655" y="30.099" smashed="yes" rot="R180">
-<attribute name="PROD_ID" value=" " x="33.655" y="30.099" size="1.778" layer="27" rot="R180" display="off"/>
-<attribute name="VALUE" x="33.655" y="28.702" size="0.6096" layer="25" font="vector" ratio="20" rot="R180" align="top-center"/>
+<element name="R2" library="SparkFun-Resistors" library_urn="urn:adsk.eagle:library:532" package="0603" package3d_urn="urn:adsk.eagle:package:39650/1" value="1k" x="33.655" y="30.099" smashed="yes" rot="R180">
+<attribute name="PROD_ID" value="RES-07856" x="33.655" y="30.099" size="1.778" layer="27" rot="R180" display="off"/>
+<attribute name="VALUE" value="1k" x="33.655" y="28.702" size="0.6096" layer="25" font="vector" ratio="20" rot="R180" align="top-center"/>
 </element>
 <element name="R3" library="SparkFun-Resistors" package="0603" value="2.0k" x="32.131" y="7.62" smashed="yes">
@@
 <attribute name="NAME" x="29.831" y="0.654" size="0.6096" layer="25" ratio="10" rot="R90"/>
 </element>
-<element name="SPK-SW" library="SparkFun-Connectors" package="1X02" value="" x="46.228" y="10.541"/>
+<element name="SPK-SW" library="SparkFun-Connectors" package="1X02" value="" x="46.228" y="10.541" smashed="yes">
+<attribute name="NAME" x="44.958" y="11.938" size="0.6096" layer="25" font="vector" ratio="20"/>
+<attribute name="VALUE" x="44.958" y="8.509" size="0.6096" layer="27" font="vector" ratio="20"/>
+</element>
 <element name="SPK-XFMR" library="trafo-xicon" library_urn="urn:adsk.eagle:library:393" package="42TL" package3d_urn="urn:adsk.eagle:package:28185/1" value="42TL016" x="42.037" y="25.4" smashed="yes">
 <attribute name="MF" value="" x="42.037" y="25.4" size="1.778" layer="27" display="off"/>
@@
 <attribute name="VALUE" x="13.97" y="29.21" size="0.6096" layer="25" font="vector" ratio="20" rot="R180" align="top-center"/>
 </element>
-<element name="R8" library="SparkFun-Resistors" library_urn="urn:adsk.eagle:library:532" package="0603" package3d_urn="urn:adsk.eagle:package:39650/1" value="100" x="34.036" y="19.05" smashed="yes">
-<attribute name="PROD_ID" value="RES-07863" x="34.036" y="19.05" size="1.778" layer="27" display="off"/>
-<attribute name="VALUE" x="34.036" y="20.447" size="0.6096" layer="25" font="vector" ratio="20" align="top-center"/>
-</element>
-<element name="R9" library="SparkFun-Resistors" library_urn="urn:adsk.eagle:library:532" package="0603" package3d_urn="urn:adsk.eagle:package:39650/1" value="100" x="37.465" y="37.846" smashed="yes" rot="R180">
-<attribute name="PROD_ID" value="RES-07863" x="37.465" y="37.846" size="1.778" layer="27" rot="R180" display="off"/>
-<attribute name="VALUE" x="37.465" y="36.449" size="0.6096" layer="25" font="vector" ratio="20" rot="R180" align="top-center"/>
+<element name="R8" library="SparkFun-Resistors" library_urn="urn:adsk.eagle:library:532" package="0603" package3d_urn="urn:adsk.eagle:package:39650/1" value="1k" x="34.036" y="19.05" smashed="yes">
+<attribute name="PROD_ID" value="RES-07856" x="34.036" y="19.05" size="1.778" layer="27" display="off"/>
+<attribute name="VALUE" value="1k" x="34.036" y="20.447" size="0.6096" layer="25" font="vector" ratio="20" align="top-center"/>
+</element>
+<element name="R9" library="SparkFun-Resistors" library_urn="urn:adsk.eagle:library:532" package="0603" package3d_urn="urn:adsk.eagle:package:39650/1" value="1k" x="37.465" y="37.846" smashed="yes" rot="R180">
+<attribute name="PROD_ID" value="RES-07856" x="37.465" y="37.846" size="1.778" layer="27" rot="R180" display="off"/>
+<attribute name="VALUE" value="1k" x="37.465" y="36.449" size="0.6096" layer="25" font="vector" ratio="20" rot="R180" align="top-center"/>
 </element>
 </elements>
@@
 </signal>
 </signals>
+<mfgpreviewcolors>
+<mfgpreviewcolor name="soldermaskcolor" color="0xC8008000"/>
+<mfgpreviewcolor name="silkscreencolor" color="0xFFFEFEFE"/>
+<mfgpreviewcolor name="backgroundcolor" color="0xFF282828"/>
+<mfgpreviewcolor name="coppercolor" color="0xFFFFBF00"/>
+<mfgpreviewcolor name="substratecolor" color="0xFF786E46"/>
+</mfgpreviewcolors>
 </board>
 </drawing>

Commit message: Updated resistor values on adapter board to be consistent with what I ended up building
Parts:
- R2: value 1k -> 120
- R8, R9: value 1k -> 100
Other:
- board text added: "120"
Changed lines of the file:
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@@
 <text x="35.56" y="6.35" size="0.6096" layer="22" rot="MR270">RX</text>
 <text x="33.02" y="6.35" size="0.6096" layer="22" rot="MR270">GND</text>
+<text x="33.655" y="31.623" size="0.6096" layer="25" font="vector" ratio="20" align="top-center">120</text>
 </plain>
 <attributes>
@@
 <attribute name="VALUE" x="48.26" y="8.255" size="0.6096" layer="25" font="vector" ratio="20" rot="R180" align="top-center"/>
 </element>
-<element name="R2" library="SparkFun-Resistors" library_urn="urn:adsk.eagle:library:532" package="0603" package3d_urn="urn:adsk.eagle:package:39650/1" value="1k" x="33.655" y="30.099" smashed="yes" rot="R180">
-<attribute name="PROD_ID" value="RES-07856" x="33.655" y="30.099" size="1.778" layer="27" rot="R180" display="off"/>
-<attribute name="VALUE" value="1k" x="33.655" y="28.702" size="0.6096" layer="25" font="vector" ratio="20" rot="R180" align="top-center"/>
+<element name="R2" library="SparkFun-Resistors" library_urn="urn:adsk.eagle:library:532" package="0603" package3d_urn="urn:adsk.eagle:package:39650/1" value="120" x="33.655" y="30.099" smashed="yes" rot="R180">
+<attribute name="PROD_ID" value=" " x="33.655" y="30.099" size="1.778" layer="27" rot="R180" display="off"/>
+<attribute name="VALUE" value=" " x="33.655" y="28.702" size="0.6096" layer="25" font="vector" ratio="20" rot="R180" align="top-center"/>
 </element>
 <element name="R3" library="SparkFun-Resistors" package="0603" value="2.0k" x="32.131" y="7.62" smashed="yes">
@@
 <attribute name="VALUE" x="13.97" y="29.21" size="0.6096" layer="25" font="vector" ratio="20" rot="R180" align="top-center"/>
 </element>
-<element name="R8" library="SparkFun-Resistors" library_urn="urn:adsk.eagle:library:532" package="0603" package3d_urn="urn:adsk.eagle:package:39650/1" value="1k" x="34.036" y="19.05" smashed="yes">
-<attribute name="PROD_ID" value="RES-07856" x="34.036" y="19.05" size="1.778" layer="27" display="off"/>
-<attribute name="VALUE" value="1k" x="34.036" y="20.447" size="0.6096" layer="25" font="vector" ratio="20" align="top-center"/>
-</element>
-<element name="R9" library="SparkFun-Resistors" library_urn="urn:adsk.eagle:library:532" package="0603" package3d_urn="urn:adsk.eagle:package:39650/1" value="1k" x="37.465" y="37.846" smashed="yes" rot="R180">
-<attribute name="PROD_ID" value="RES-07856" x="37.465" y="37.846" size="1.778" layer="27" rot="R180" display="off"/>
-<attribute name="VALUE" value="1k" x="37.465" y="36.449" size="0.6096" layer="25" font="vector" ratio="20" rot="R180" align="top-center"/>
+<element name="R8" library="SparkFun-Resistors" library_urn="urn:adsk.eagle:library:532" package="0603" package3d_urn="urn:adsk.eagle:package:39650/1" value="100" x="34.036" y="19.05" smashed="yes">
+<attribute name="PROD_ID" value="RES-12438" x="34.036" y="19.05" size="1.778" layer="27" display="off"/>
+<attribute name="VALUE" value="100" x="34.036" y="20.447" size="0.6096" layer="25" font="vector" ratio="20" align="top-center"/>
+</element>
+<element name="R9" library="SparkFun-Resistors" library_urn="urn:adsk.eagle:library:532" package="0603" package3d_urn="urn:adsk.eagle:package:39650/1" value="100" x="37.465" y="37.846" smashed="yes" rot="R180">
+<attribute name="PROD_ID" value="RES-12438" x="37.465" y="37.846" size="1.778" layer="27" rot="R180" display="off"/>
+<attribute name="VALUE" value="100" x="37.465" y="36.449" size="0.6096" layer="25" font="vector" ratio="20" rot="R180" align="top-center"/>
 </element>
 </elements>
@@
 <contactref element="C18" pad="1"/>
 <contactref element="FB1" pad="1"/>
-<contactref element="R2" pad="2"/>
 <wire x1="18.249" y1="30.607" x2="16.002" y2="32.854" width="0.1524" layer="1"/>
 <wire x1="16.002" y1="32.854" x2="16.002" y2="34.29" width="0.1524" layer="1"/>
@@
 <wire x1="13.12" y1="31.408" x2="13.12" y2="30.607" width="0.1524" layer="1"/>
 <wire x1="13.12" y1="30.607" x2="11.391" y2="30.607" width="0.1524" layer="1"/>
+<contactref element="R2" pad="2"/>
 </signal>
 <signal name="HANDSET-SPK">
@@
 <contactref element="Q2" pad="3"/>
 <contactref element="C1" pad="+"/>
-<contactref element="R2" pad="1"/>
 <contactref element="R7" pad="S"/>
 <wire x1="34.505" y1="30.099" x2="34.505" y2="33.186" width="0.1524" layer="1"/>
@@
 <wire x1="22.352" y1="34.544" x2="26.035" y2="38.227" width="0.1524" layer="1"/>
 <wire x1="26.035" y1="38.227" x2="27.94" y2="38.227" width="0.1524" layer="1"/>
+<contactref element="R2" pad="1"/>
 </signal>
 <signal name="N$2">
